File: nrf2rfm69.sch (KiCad schematic (older format))
At the start: 4 parts, among them P1 CONN_01X01, U1 RFM69HW, U2 NRF24L01

Commit message: Shrinked pcb a bit, and created panel layout for dirtypcb's
Parts:
- P1: footprint Socket_Strips:Socket_Strip_Angled_1x01 -> Socket_Strips:Socket_Strip_Straight_1x01
Changed lines of the file:
@@
 F 0 "P1" H 6050 3750 50  0000 C CNN
 F 1 "CONN_01X01" V 6150 3650 50  0000 C CNN
-F 2 "Socket_Strips:Socket_Strip_Angled_1x01" H 6050 3650 50  0001 C CNN
+F 2 "Socket_Strips:Socket_Strip_Straight_1x01" H 6050 3650 50  0001 C CNN
 F 3 "" H 6050 3650 50  0000 C CNN
 	1    6050 3650
@@
 07 00 85 88 3B 00 28 44 DC 01 40 21 E2 0E 00 0A 11 77 00 50 88 B8 03 80 42 C4 1D 00 14 22 EE 00
 A0 10 71 07 00 85 88 3B 00 28 F4 2F 6E 0E 73 66 69 F5 31 42 00 00 00 00 49 45 4E 44 AE 42 60 82
-00
+58
 EndData
 $EndBitmap
